Commit message: Rotated lidar mesh

File: magni_description/urdf/sensors/rplidar.xacro (robot description, xacro)
@@ -11,5 +11,5 @@
   <link name="${name}">
     <visual>
-      <origin xyz="0 0 -0.03" rpy="0 0 ${pi/2}" />
+      <origin xyz="0 0 -0.03" rpy="0 0 ${-pi/2}" />
       <geometry>
         <mesh filename="package://magni_description/meshes/sensors/RPLIDAR.stl" />
@@ -28,5 +28,5 @@
       <pose>0 0 0 0 0 0</pose>
       <visualize>false</visualize>
-      <update_rate>20</update_rate>
+      <update_rate>10</update_rate>
       <ray>
         <scan>
