Commit message: add rplidar

File: magni_description/urdf/magni.urdf.xacro (robot description, xacro)
@@ -19,4 +19,5 @@
   <xacro:include filename="$(find magni_description)/urdf/sensors/raspi_camera.xacro" />
   <xacro:include filename="$(find magni_description)/urdf/sensors/ur50_lidar.xacro" />
+  <xacro:include filename="$(find magni)/urdf/sensors/rplidar.xacro" />
   <!-- Robot base_link -->
   <link name="base_link">
@@ -212,10 +213,7 @@
   </xacro:if>
   <!-- Define Lidar -->
-  <xacro:if value="${lidar_extrinsics_file != ''}">
-    <xacro:property name="lidar_extrinsics" value="${load_yaml(lidar_extrinsics_file)}"/>
-    <xacro:ur50_lidar name="laser" connected_to="base_link">
-      <origin xyz="${lidar_extrinsics['x']} ${lidar_extrinsics['y']} ${lidar_extrinsics['z']}"
-        rpy="${lidar_extrinsics['roll']} ${lidar_extrinsics['pitch']} ${lidar_extrinsics['yaw']}"/>
-    </xacro:ur50_lidar>
-  </xacro:if>
+  <xacro:rplidar name="laser" connected_to="base_link">
+      <origin xyz="0.09 0 0.21"
+        rpy="0 0 0"/>
+  </xacro:rplidar>
 </robot>

Commit message: oak-d camera on urdf

File: magni_description/urdf/magni.urdf.xacro (robot description, xacro)
@@ -20,4 +20,5 @@
   <xacro:include filename="$(find magni_description)/urdf/sensors/ur50_lidar.xacro" />
   <xacro:include filename="$(find magni_description)/urdf/sensors/rplidar.xacro" />
+  <xacro:include filename="$(find magni_description)/urdf/sensors/oak-d.xacro" />
   <!-- Robot base_link -->
   <link name="base_link">
@@ -212,4 +213,8 @@
     </xacro:raspi_camera>
   </xacro:if>
+  <xacro:oak-d name="oakd" connected_to="base_link">
+    <origin xyz="0.125 0 0.093"
+      rpy="0 0 0" />
+  </xacro:oak-d>
   <!-- Define Lidar -->
   <xacro:rplidar name="laser" connected_to="base_link">
